File: fauxmo-smd.sch (EAGLE design)
At the start: 22 parts, among them J1 POWERJACKPTH, Q1 IRLB8721PBF, Q2 IRLB8721PBF, Q3 IRLB8721PBF, Q4 IRLB8721PBF

Commit message: Add files via upload
Connections:
- net BLUE: now also X1.GPIO12; no longer X1.GPIO14
- net GREEN: now also X1.GPIO14; no longer X1.GPIO13
- net RED: now also X1.GPIO16; no longer X1.GPIO12
- net WHITE: now also X1.GPIO13; no longer X1.GPIO16
Changed lines of the file:
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@@
 <?xml version="1.0" encoding="utf-8"?>
 <!DOCTYPE eagle SYSTEM "eagle.dtd">
-<eagle version="8.5.1">
+<eagle version="8.5.0">
 <drawing>
 <settings>
@@
 </busses>
 <nets>
-<net name="RED" class="0">
+<net name="BLUE" class="0">
 <segment>
 <pinref part="X1" gate="G$1" pin="GPIO12"/>
@@
 </segment>
 <segment>
-<pinref part="Q4" gate="G$1" pin="G"/>
-<wire x1="106.68" y1="66.04" x2="104.14" y2="63.5" width="0.1524" layer="91"/>
-<label x="104.14" y="63.5" size="1.27" layer="95" rot="R180" xref="yes"/>
-</segment>
-</net>
-<net name="GREEN" class="0">
+<pinref part="Q3" gate="G$1" pin="G"/>
+<wire x1="88.9" y1="66.04" x2="86.36" y2="66.04" width="0.1524" layer="91"/>
+<label x="86.36" y="66.04" size="1.778" layer="95" rot="R180"/>
+</segment>
+</net>
+<net name="WHITE" class="0">
 <segment>
 <pinref part="X1" gate="G$1" pin="GPIO13"/>
@@
 </segment>
 <segment>
-<pinref part="Q2" gate="G$1" pin="G"/>
-<wire x1="127" y1="66.04" x2="124.46" y2="63.5" width="0.1524" layer="91"/>
-<label x="124.46" y="63.5" size="1.27" layer="95" rot="R180" xref="yes"/>
-</segment>
-</net>
-<net name="BLUE" class="0">
+<pinref part="Q1" gate="G$1" pin="G"/>
+<wire x1="71.12" y1="66.04" x2="68.58" y2="66.04" width="0.1524" layer="91"/>
+<label x="68.58" y="66.04" size="1.778" layer="95" rot="R180"/>
+</segment>
+</net>
+<net name="GREEN" class="0">
 <segment>
 <pinref part="X1" gate="G$1" pin="GPIO14"/>
@@
 </segment>
 <segment>
-<pinref part="Q3" gate="G$1" pin="G"/>
-<wire x1="88.9" y1="66.04" x2="86.36" y2="63.5" width="0.1524" layer="91"/>
-<label x="86.36" y="63.5" size="1.27" layer="95" rot="R180" xref="yes"/>
-</segment>
-</net>
-<net name="WHITE" class="0">
+<pinref part="Q2" gate="G$1" pin="G"/>
+<wire x1="127" y1="66.04" x2="124.46" y2="66.04" width="0.1524" layer="91"/>
+<label x="124.46" y="66.04" size="1.778" layer="95" rot="R180"/>
+</segment>
+</net>
+<net name="RED" class="0">
 <segment>
 <pinref part="X1" gate="G$1" pin="GPIO16"/>
@@
 </segment>
 <segment>
-<pinref part="Q1" gate="G$1" pin="G"/>
-<wire x1="71.12" y1="66.04" x2="68.58" y2="63.5" width="0.1524" layer="91"/>
-<label x="68.58" y="63.5" size="1.27" layer="95" rot="R180" xref="yes"/>
-</segment>
-</net>
+<pinref part="Q4" gate="G$1" pin="G"/>
+<wire x1="106.68" y1="66.04" x2="104.14" y2="66.04" width="0.1524" layer="91"/>
+<label x="104.14" y="66.04" size="1.778" layer="95" rot="R180"/>
+</segment>
+</net>
